File: CPU_meter.sch (KiCad schematic (older format))
At the start: 22 parts, among them IC1 ATMEGA328P-P, SW1 SPST, U1 74HC595, U2 74HC595, U3 74HC595, U4 74HC595, U5 74HC595, U6 LM7805, Y1 16.00 MHz

Commit message: Finalized the board layout for first prototype run!
Parts:
- added P1, P4: CONN_01X02, Terminal_Blocks:TerminalBlock_Pheonix_MPT-2.54mm_2pol, symbol CONN_01X02
- added P2: CONN_01X14, Connect:IDC_Header_Straight_14pins, symbol CONN_01X14
- added P3: CONN_01X02, Terminal_Blocks:TerminalBlock_Pheonix_PT-3.5mm_2pol, symbol CONN_01X02
- IC1: value ATMEGA328P-P -> ATMEGA328P
- U6: footprint TO_SOT_Packages_THT:TO-220_Neutral123_Horizontal_Reverse -> Resistor array:TO-220_Neutral123_Horizontal_Reverse
Connections:
- net +12V: now also P3.1 (P1)
- net GND: now also P3.2 (P2), P4.2 (P2)
- net VCC: now also P4.1 (P1)
- net at IC1.11 ((PCINT21/OC0B/T1)PD5): now also IC1.24 ((PCINT9/ADC1)PC1), P2.4 (P4), P2.9 (P9)
- net at IC1.12 ((PCINT22/OC0A/AIN0)PD6): now also P2.5 (P5)
- net at IC1.15 ((PCINT1/OC1A)PB1): now also P2.6 (P6)
- net at IC1.19 ((PCINT5/SCK)PB5): now also P2.7 (P7)
- net at IC1.2 ((PCINT16/RXD)PD0): now also IC1.27 ((PCINT12/SDA/ADC4)PC4), P1.1 (P1), P2.12 (P12)
- net at IC1.21 (AREF): now also P2.14 (P14)
- net at IC1.23 ((PCINT8/ADC0)PC0): now also P2.8 (P8)
- net at IC1.25 ((PCINT10/ADC2)PC2): now also P2.10 (P10)
- net at IC1.26 ((PCINT11/ADC3)PC3): now also P2.11 (P11)
- net at IC1.28 ((PCINT13/SCL/ADC5)PC5): now also P2.13 (P13)
- net at IC1.3 ((PCINT17/TXD)PD1): now also P1.2 (P2)
- net at IC1.4 ((PCINT18/INT0)PD2): now also P2.1 (P1)
- net at IC1.5 ((PCINT19/OC2B/INT1)PD3): now also P2.2 (P2)
- net at IC1.6 ((PCINT20/XCK/T0)PD4): now also P2.3 (P3)
