File: CPU_meter.kicad_pcb (KiCad board)
At the start: 4 copper layers, 25 parts, among them IC1 ATMEGA328P-P, SW1 SPST, U1 74HC595, U2 74HC595, U3 74HC595, U4 74HC595, U5 74HC595, U6 LM7805, Y1 16.00 MHz

Commit message: Finalized the board layout for first prototype run!
Parts:
- removed the REF** at (115.6, 124.5)
- removed the REF** at (115.6, 139.7)
- removed the REF** at (115.6, 132.1)
- added P1: RX TX, Terminal_Blocks:TerminalBlock_Pheonix_MPT-2.54mm_2pol, F.Cu at (160.5, 81.9)
- added P2: CONN_01X14, Connect:IDC_Header_Straight_14pins, F.Cu at (165.6, 117.4)
- added P3: GND VIN, Terminal_Blocks:TerminalBlock_Pheonix_PT-3.5mm_2pol, F.Cu at (100.8, 76.8)
- added P4: +5V GND, Terminal_Blocks:TerminalBlock_Pheonix_MPT-2.54mm_2pol, F.Cu at (160.5, 75.5)
- added REF**: Mounting Hole, Mounting_Holes:MountingHole_2.7mm_M2.5_ISO7380_Pad, F.Cu at (164.3, 127.6)
- added REF**: Mounting Hole, Mounting_Holes:MountingHole_2.7mm_M2.5_ISO7380_Pad, F.Cu at (163.1, 92.0)
- added REF**: Mounting Hole, Mounting_Holes:MountingHole_2.7mm_M2.5_ISO7380_Pad, F.Cu at (156.7, 140.3)
- added REF**: MountingHole_2.7mm_M2.5, Mounting_Holes:MountingHole_2.7mm_M2.5_ISO7380_Pad, F.Cu at (100.8, 71.7)
- added REF**: Mounting Hole, Mounting_Holes:MountingHole_2.7mm_M2.5_ISO7380_Pad, F.Cu at (152.9, 86.9)
- added REF**: Mounting Hole, Mounting_Holes:MountingHole_2.7mm_M2.5_ISO7380_Pad, F.Cu at (95.8, 116.1)
- C2: moved to F.Cu
- IC1: value ATMEGA328P-P -> ATMEGA328P; moved to F.Cu
- U6: footprint TO_SOT_Packages_THT:TO-220_Neutral123_Horizontal_Reverse -> Resistor array:TO-220_Neutral123_Horizontal_Reverse
- moved C1 67.1 mm to (103.5, 87.6)
- moved C2 66.9 mm to (148.0, 77.5), turned to 90 degrees
- moved Y1 50.8 mm to (145.4, 86.4), turned to 90 degrees
- moved RR4 49.6 mm to (126.4, 71.1)
- moved U2 49.0 mm to (112.4, 111.8)
- moved BAR4 44.8 mm to (126.4, 77.5)
- moved U5 43.7 mm to (122.6, 76.2)
- moved RR3 42.5 mm to (126.4, 88.9)
- moved U3 41.1 mm to (101.0, 94.0), turned to 270 degrees
- moved SW1 40.8 mm to (107.3, 77.5)
- moved BAR3 37.8 mm to (126.4, 95.2)
- moved RR2 37.8 mm to (126.4, 106.7)
- moved C3 32.8 mm to (104.8, 115.6)
- moved IC1 31.5 mm to (145.4, 102.9), turned to 0 degrees
- moved RR1 31.0 mm to (126.4, 124.5)
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Routing:
- net VCC: track 95.8 -> 305.2 mm, vias 0 -> 8
- net Net-(IC1-Pad17): track 0.00 -> 206.5 mm, vias 0 -> 2
- net GND: track 128.7 -> 329.8 mm, vias 0 -> 14
- net Net-(IC1-Pad18): track 0.00 -> 181.9 mm, vias 0 -> 3
- net Net-(IC1-Pad1): track 0.00 -> 140.6 mm, vias 0 -> 1
- net +12V: track 0.00 -> 97.1 mm
- net Net-(U1-Pad9): track 10.2 -> 89.8 mm, vias 0 -> 6
- net Net-(C1-Pad1): track 9.84 -> 83.9 mm, vias 0 -> 1
- net Net-(BAR1-Pad9): track 4.86 -> 78.9 mm, vias 0 -> 4
- net Net-(IC1-Pad16): track 0.00 -> 68.4 mm, vias 0 -> 4
- net Net-(C2-Pad1): track 0.00 -> 60.9 mm
- net Net-(BAR2-Pad7): track 0.00 -> 55.0 mm, vias 0 -> 4
- net Net-(BAR2-Pad8): track 0.00 -> 52.7 mm, vias 0 -> 3
- net Net-(IC1-Pad5): track 0.00 -> 52.6 mm, vias 0 -> 7
- net Net-(BAR3-Pad8): track 58.1 -> 6.66 mm
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Other:
- copper layers 4 -> 2
